Commit message: Adding moving object

File: ufn_code/src/unconstrained_navigation_fetch_mapping/launch/objects/bean_box.urdf (robot description, URDF)
Before this commit: robot bean_box, 2 links, 1 joints
Links:
- link box_base: geometry collision mesh filename=package://unconstrained_navigation_fetch_mapping/launch/obj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; visual mesh filename=package://unconstrained_navigation_fetch_mapping/launch/obj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
- link box_lid: geometry collision mesh filename=package://unconstrained_navigation_fetch_mapping/launch/obj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; visual mesh filename=package://unconstrained_navigation_fetch_mapping/launch/obj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

File: ufn_code/src/unconstrained_navigation_fetch_mapping/launch/objects/kitchen_counter.urdf (robot description, URDF)
Before this commit: robot counter, 1 links, 0 joints
Links:
- link kitchen_counter: geometry collision mesh filename=package://unconstrained_navigation_fetch_mapping/launch/obj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; visual mesh filename=package://unconstrained_navigation_fetch_mapping/launch/obj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
